File: doc/hardware/main-board/sd-mux.sch (KiCad schematic (older format))
At the start: 48 parts, among them J1 USDCARD, P1 USB_OTG, P10 MKDS 1,5/3, P2 629105136821, P3 61400416021, P4 61400416021, P5 IDC_02X04, P6 IDC_02X04, P7 MKDS 1,5/3, P8 CONN_02X02, P9 CONN_02X02, Q1 IRF7606PBF, Q2 IRF7606PBF, Q3 IRF7606PBF, Q4 IRF7606PBF, Q5 2N7002, Q6 2N7002, Q7 IRF7606PBF, Q8 IRF7606PBF, U1 TS3USB30EDGSR, U2 FT245RL, U3 74AHC1G14, U4 TS3A27518E, U5 74AHC1G14

Commit message: Fix power supply connection of USB switch inverter
Power supply pin of U5 was connected to 3.3V. Q8, driven from this
inverter, couldn't be fully closed as maximum output voltage from
the inverter was 3.3V. Now, the inverter, is connected to VCC pin
of USB connector which gives 5V.

Change-Id: Ibed75765ea8cbc2727066d6a498a3396a2d3c404
Parts:
- P1, P2: symbol USB_OTG -> USB_OTG-RESCUE-sd-mux
- P3, P4: symbol USB_A -> USB_A-RESCUE-sd-mux
Changed lines of the file:
@@
 EESchema Schematic File Version 2
+LIBS:sd-mux-rescue
 LIBS:sd-relay
 LIBS:power
@@
 Sheet 1 1
 Title "sd-mux"
-Date "2016-02-26"
-Rev "2"
+Date "2016-11-14"
+Rev "2.1"
 Comp "SRPOL"
 Comment1 "Author: Adam Malinowski <a.malinowsk2@partner.samsung.com>"
@@
 $EndComp
 $Comp
-L USB_OTG P1
+L USB_OTG-RESCUE-sd-mux P1
 U 1 1 55F72E39
 P 850 1550
@@
 NoConn ~ 12500 8900
 $Comp
-L VDD #PWR024
+L VDD #PWR023
 U 1 1 55F71867
 P 9200 10200
-F 0 "#PWR024" H 9200 10050 50  0001 C CNN
+F 0 "#PWR023" H 9200 10050 50  0001 C CNN
 F 1 "VDD" H 9200 10350 50  0000 C CNN
 F 2 "" H 9200 10200 60  0000 C CNN
@@
 $EndComp
 $Comp
-L VDD #PWR025
+L VDD #PWR024
 U 1 1 55F7196F
 P 9550 10200
-F 0 "#PWR025" H 9550 10050 50  0001 C CNN
+F 0 "#PWR024" H 9550 10050 50  0001 C CNN
 F 1 "VDD" H 9550 10350 50  0000 C CNN
 F 2 "" H 9550 10200 60  0000 C CNN
@@
 $EndComp
 $Comp
-L USB_OTG P2
+L USB_OTG-RESCUE-sd-mux P2
 U 1 1 55FB52CC
 P 1600 6450
@@
 $EndComp
 $Comp
-L GND #PWR026
+L GND #PWR025
 U 1 1 55FB52D2
 P 2000 6750
-F 0 "#PWR026" H 2000 6500 50  0001 C CNN
+F 0 "#PWR025" H 2000 6500 50  0001 C CNN
 F 1 "GND" H 2000 6600 50  0000 C CNN
 F 2 "" H 2000 6750 60  0000 C CNN
@@
 $EndComp
 $Comp
-L GND #PWR027
+L GND #PWR026
 U 1 1 55FB52E4
 P 1500 7600
-F 0 "#PWR027" H 1500 7350 50  0001 C CNN
+F 0 "#PWR026" H 1500 7350 50  0001 C CNN
 F 1 "GND" H 1500 7450 50  0000 C CNN
 F 2 "" H 1500 7600 60  0000 C CNN
@@
 NoConn ~ 1900 6550
 $Comp
-L USB_A P3
+L USB_A-RESCUE-sd-mux P3
 U 1 1 55FB5556
 P 6200 6450
@@
 $EndComp
 $Comp
-L GND #PWR028
+L GND #PWR027
 U 1 1 55FB5853
 P 6300 7450
-F 0 "#PWR028" H 6300 7200 50  0001 C CNN
+F 0 "#PWR027" H 6300 7200 50  0001 C CNN
 F 1 "GND" H 6300 7300 50  0000 C CNN
 F 2 "" H 6300 7450 60  0000 C CNN
@@
 $EndComp
 $Comp
-L GND #PWR029
+L GND #PWR028
 U 1 1 55FB5AC1
 P 5800 6650
-F 0 "#PWR029" H 5800 6400 50  0001 C CNN
+F 0 "#PWR028" H 5800 6400 50  0001 C CNN
 F 1 "GND" H 5800 6500 50  0000 C CNN
 F 2 "" H 5800 6650 60  0000 C CNN
@@
 $EndComp
 $Comp
-L USB_A P4
+L USB_A-RESCUE-sd-mux P4
 U 1 1 55FC51B0
 P 6200 8000
@@
 $EndComp
 $Comp
-L GND #PWR030
+L GND #PWR029
 U 1 1 55FC51C2
 P 6300 9000
-F 0 "#PWR030" H 6300 8750 50  0001 C CNN
+F 0 "#PWR029" H 6300 8750 50  0001 C CNN
 F 1 "GND" H 6300 8850 50  0000 C CNN
 F 2 "" H 6300 9000 60  0000 C CNN
@@
 $EndComp
 $Comp
-L GND #PWR031
+L GND #PWR030
 U 1 1 55FC51D2
 P 5800 8200
-F 0 "#PWR031" H 5800 7950 50  0001 C CNN
+F 0 "#PWR030" H 5800 7950 50  0001 C CNN
 F 1 "GND" H 5800 8050 50  0000 C CNN
 F 2 "" H 5800 8200 60  0000 C CNN
@@
 $EndComp
 $Comp
-L GND #PWR032
+L GND #PWR031
 U 1 1 55FD1DB0
 P 3550 7300
-F 0 "#PWR032" H 3550 7050 50  0001 C CNN
+F 0 "#PWR031" H 3550 7050 50  0001 C CNN
 F 1 "GND" H 3550 7150 50  0000 C CNN
 F 2 "" H 3550 7300 60  0000 C CNN
@@
 $EndComp
 $Comp
-L VDD #PWR033
+L VDD #PWR032
 U 1 1 55FD2ADD
 P 3550 7000
-F 0 "#PWR033" H 3550 6850 50  0001 C CNN
+F 0 "#PWR032" H 3550 6850 50  0001 C CNN
 F 1 "VDD" H 3550 7150 50  0000 C CNN
 F 2 "" H 3550 7000 60  0000 C CNN
@@
 $EndComp
 $Comp
-L GND #PWR034
+L GND #PWR033
 U 1 1 55FD3482
 P 2250 7300
-F 0 "#PWR034" H 2250 7050 50  0001 C CNN
+F 0 "#PWR033" H 2250 7050 50  0001 C CNN
 F 1 "GND" H 2250 7150 50  0000 C CNN
 F 2 "" H 2250 7300 60  0000 C CNN
@@
 	10950 8700 10750 8700
 $Comp
-L +3V3 #PWR035
+L +3V3 #PWR034
 U 1 1 56426AA3
 P 2200 2150
-F 0 "#PWR035" H 2200 2000 50  0001 C CNN
+F 0 "#PWR034" H 2200 2000 50  0001 C CNN
 F 1 "+3V3" H 2200 2290 50  0000 C CNN
 F 2 "" H 2200 2150 60  0000 C CNN
@@
 Connection ~ 2300 2200
 $Comp
-L +3V3 #PWR036
+L +3V3 #PWR035
 U 1 1 564287DB
 P 13400 6000
-F 0 "#PWR036" H 13400 5850 50  0001 C CNN
+F 0 "#PWR035" H 13400 5850 50  0001 C CNN
 F 1 "+3V3" H 13400 6140 50  0000 C CNN
 F 2 "" H 13400 6000 60  0000 C CNN
@@
 $EndComp
 $Comp
-L +3V3 #PWR037
+L +3V3 #PWR036
 U 1 1 5642ADDD
 P 8500 10200
-F 0 "#PWR037" H 8500 10050 50  0001 C CNN
+F 0 "#PWR036" H 8500 10050 50  0001 C CNN
 F 1 "+3V3" H 8500 10340 50  0000 C CNN
 F 2 "" H 8500 10200 60  0000 C CNN
@@
 	13050 2800 12950 2800
 $Comp
-L +3V3 #PWR038
+L +3V3 #PWR037
 U 1 1 56509DD4
 P 11150 2850
-F 0 "#PWR038" H 11150 2700 50  0001 C CNN
+F 0 "#PWR037" H 11150 2700 50  0001 C CNN
 F 1 "+3V3" H 11150 2990 50  0000 C CNN
 F 2 "" H 11150 2850 60  0000 C CNN
@@
 $EndComp
 $Comp
-L GND #PWR039
+L GND #PWR038
 U 1 1 5650C07E
 P 12150 2300
-F 0 "#PWR039" H 12150 2050 50  0001 C CNN
+F 0 "#PWR038" H 12150 2050 50  0001 C CNN
 F 1 "GND" H 12150 2150 50  0000 C CNN
 F 2 "" H 12150 2300 60  0000 C CNN
@@
 $EndComp
 $Comp
-L GND #PWR040
+L GND #PWR039
 U 1 1 5650C4C2
 P 12150 3350
-F 0 "#PWR040" H 12150 3100 50  0001 C CNN
+F 0 "#PWR039" H 12150 3100 50  0001 C CNN
 F 1 "GND" H 12150 3200 50  0000 C CNN
 F 2 "" H 12150 3350 60  0000 C CNN
@@
 $EndComp
 $Comp
-L GND #PWR041
+L GND #PWR040
 U 1 1 565228EA
 P 4500 8750
-F 0 "#PWR041" H 4500 8500 50  0001 C CNN
+F 0 "#PWR040" H 4500 8500 50  0001 C CNN
 F 1 "GND" H 4500 8600 50  0000 C CNN
 F 2 "" H 4500 8750 60  0000 C CNN
@@
 $EndComp
 $Comp
-L VDD #PWR043
+L VDD #PWR041
 U 1 1 56534188
 P 1650 8100
-F 0 "#PWR043" H 1650 7950 50  0001 C CNN
+F 0 "#PWR041" H 1650 7950 50  0001 C CNN
 F 1 "VDD" H 1650 8250 50  0000 C CNN
 F 2 "" H 1650 8100 60  0000 C CNN
@@
 Connection ~ 1650 8500
 $Comp
-L +3V3 #PWR044
+L +3V3 #PWR042
 U 1 1 56535F81
 P 8850 10200
-F 0 "#PWR044" H 8850 10050 50  0001 C CNN
+F 0 "#PWR042" H 8850 10050 50  0001 C CNN
 F 1 "+3V3" H 8850 10340 50  0000 C CNN
 F 2 "" H 8850 10200 60  0000 C CNN
@@
 $EndComp
 $Comp
-L +3V3 #PWR?
+L +3V3 #PWR043
 U 1 1 5653649E
 P 11350 1750
-F 0 "#PWR?" H 11350 1600 50  0001 C CNN
+F 0 "#PWR043" H 11350 1600 50  0001 C CNN
 F 1 "+3V3" H 11350 1890 50  0000 C CNN
 F 2 "" H 11350 1750 60  0000 C CNN
